File: PCB/carrier.kicad_pcb (KiCad board)
At the start: 6 copper layers, 69.6 x 46.1 mm, 98 parts, among them J1 SODIMM-260_Split, J2 Micro_SD_Card_Det2, Q2 BSS138, Q3 BSS138, Q4 BC817-40, Q5 BSS138, SW1 SW_DIP_x04, U1 SN74LVC8T245, U2 SN74LVC8T245, U3 SN74LVC8T245, U4 RT9742GGJ5

Commit message: updated 2
Parts:
- added C1: 0.1uF, Capacitor_SMD:C_0402_1005Metric, F.Cu at (212.3, 81.0)
- added C11: 10uF, Capacitor_SMD:C_0603_1608Metric, F.Cu at (198.5, 89.5)
- added C2: 0.1uF, Capacitor_SMD:C_0402_1005Metric, F.Cu at (212.3, 82.9)
- added C20: 10uF, Capacitor_SMD:C_0603_1608Metric, F.Cu at (198.5, 92.0)
- added C4: 0.1uF, Capacitor_SMD:C_0402_1005Metric, F.Cu at (212.3, 84.9)
- added C5: 0.1uF, Capacitor_SMD:C_0402_1005Metric, F.Cu at (212.3, 86.9)
- added C6: 0.1uF, Capacitor_SMD:C_0402_1005Metric, F.Cu at (212.3, 88.8)
- added C7: 1uF, Capacitor_SMD:C_0402_1005Metric, F.Cu at (212.3, 90.8)
- added Q2: BSS138, Package_TO_SOT_SMD:SOT-23-3, F.Cu at (208.3, 82.2)
- added Q3: BSS138, Package_TO_SOT_SMD:SOT-23-3, F.Cu at (208.3, 86.6)
- added Q4: BC817-40, Package_TO_SOT_SMD:SOT-323_SC-70, F.Cu at (202.5, 89.9)
- added Q5: BSS138, Package_TO_SOT_SMD:SOT-23-3, F.Cu at (208.3, 91.1)
- added R1: 330, Resistor_SMD:R_0402_1005Metric, F.Cu at (207.2, 61.0)
- added R10: 10K, Resistor_SMD:R_0402_1005Metric, F.Cu at (207.2, 63.0)
- added R11: 10K, Resistor_SMD:R_0402_1005Metric, F.Cu at (207.2, 65.0)
- added R12: 10K, Resistor_SMD:R_0402_1005Metric, F.Cu at (207.2, 67.0)
- added R13: 10K, Resistor_SMD:R_0402_1005Metric, F.Cu at (207.2, 69.0)
- added R14: 12K, Resistor_SMD:R_0402_1005Metric, F.Cu at (207.2, 70.9)
- added R15: 330, Resistor_SMD:R_0402_1005Metric, F.Cu at (210.1, 61.0)
- added R16: 10K, Resistor_SMD:R_0402_1005Metric, F.Cu at (210.1, 63.0)
- added R17: 10K, Resistor_SMD:R_0402_1005Metric, F.Cu at (210.1, 65.0)
- added R18: 10K, Resistor_SMD:R_0402_1005Metric, F.Cu at (210.1, 67.0)
- added R19: 10K, Resistor_SMD:R_0402_1005Metric, F.Cu at (210.1, 69.0)
- added R20: 10K, Resistor_SMD:R_0402_1005Metric, F.Cu at (210.1, 70.9)
- added R21: 10K, Resistor_SMD:R_0402_1005Metric, F.Cu at (213.0, 61.0)
- added R24: 10K, Resistor_SMD:R_0402_1005Metric, F.Cu at (213.0, 63.0)
- added R25: 10K, Resistor_SMD:R_0402_1005Metric, F.Cu at (213.0, 65.0)
- added SD_PWR1: TestPoint_Small, TestPoint:TestPoint_Pad_D1.0mm, F.Cu at (148.5, 67.0)
- added TP1: RTC Test, TestPoint:TestPoint_Pad_D1.0mm, F.Cu at (190.5, 88.2)
- added TP2: Sleep Status Output, TestPoint:TestPoint_Pad_D1.0mm, F.Cu at (190.5, 91.2)
- moved D1 0.48 mm to (165.0, 59.5)
- moved J2 0.38 mm to (161.0, 70.0)
- moved SW1 0.19 mm to (103.6, 65.7)
