File: PCB/carrier.kicad_pcb (KiCad board)
At the start: 6 copper layers, 69.6 x 46.1 mm, 122 parts, among them J1 SODIMM-260_Split, J2 Micro_SD_Card_Det2, Q2 BSS138, Q3 BSS138, Q4 BC817-40, Q5 BSS138, SW1 SW_DIP_x04, U1 SN74LVC8T245, U2 SN74LVC8T245, U3 SN74LVC8T245, U4 RT9742GGJ5

Commit message: Add USB2514B hub and ECS crystal libraries, fix broken footprint/symbol links
USB2514B's placed symbol referenced a typo'd library nickname
(USBB2514B_M2) that didn't match the registered USB2514B library, and its
footprint field had the same mismatch. The ECS-240-18-33Q-DS crystal had no
symbol library registered at all and was pointing at a generic built-in
Oscillator footprint instead of its real land pattern. Added the missing
ECS library files, registered both libraries with ${KIPRJMOD}-relative
paths, and corrected the lib_id/footprint references in the schematic.

Co-Authored-By: Claude Sonnet 5 <noreply@anthropic.com>
Parts:
- added C21: 0.1uF, Capacitor_SMD:C_0402_1005Metric, F.Cu at (62.9, 74.0)
- added Y1: ECS-240-18-33Q-DS, Oscillator:Oscillator_SMD_ECS_2520MV-xxx-xx-4Pin_2.5x2.0mm, F.Cu at (55.9, 79.7)
- C12, C16, C8, C9: value 1uF -> 0.1uF
- R22, R23: value 0 -> 10K
- U1: value SN74LVC8T245 -> USB2514B/M2; footprint Package_SO:TSSOP-24_4.4x5mm_P0.4mm -> USB2514B_M2:SQFN36_6X6_MCH
- moved C1 44.9 mm to (104.0, 74.0)
- moved C2 44.9 mm to (104.0, 76.0)
- moved C4 44.9 mm to (104.0, 77.9)
- moved C5 44.9 mm to (104.0, 79.9)
- moved C6 44.9 mm to (104.0, 81.9)
- moved C7 44.9 mm to (104.0, 83.8)
- moved U1 43.7 mm to (77.5, 79.5)
- moved R10 20.0 mm to (74.0, 61.0)
- moved R11 20.0 mm to (74.0, 63.0)
- moved R12 20.0 mm to (74.0, 65.0)
- moved R13 20.0 mm to (74.0, 67.0)
- moved R14 20.0 mm to (74.0, 69.0)
- moved R15 20.0 mm to (76.9, 59.0)
- moved R16 20.0 mm to (76.9, 61.0)
- moved R17 20.0 mm to (76.9, 63.0)
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Connections:
- C12 pad 1: GND -> +3V3
- C12 pad 2: +3V3 -> GND
- C14 pad 1: GND -> +3V3
- C14 pad 2: +3V3 -> GND
- C16 pad 1: +1V8 -> Net-(U1-CRFILT)
- C3 pad 1: GND -> +3V3
- C3 pad 2: +1V8 -> GND
- C8 pad 1: GND -> +3V3
- C8 pad 2: +1V8 -> GND
- J1 pad 104: SPI-1_MOSI_1V8 -> unconnected-(J1-Pad104)
- J1 pad 106: SPI-1_CLK_1V8 -> unconnected-(J1-Pad106)
- J1 pad 108: SPI-1_MISO_1V8 -> unconnected-(J1-Pad108)
- J1 pad 109: USB3-0-DN -> unconnected-(J1-Pad109)
- J1 pad 110: SPI-1_CS0_1V8 -> unconnected-(J1-Pad110)
- J1 pad 111: USB3-0-DP -> unconnected-(J1-Pad111)
- J1 pad 112: SPI-1_CS1_1V8 -> unconnected-(J1-Pad112)
- J1 pad 114: CSI-0_PWDN -> unconnected-(J1-Pad114)
- J1 pad 115: USB3-1-DN -> unconnected-(J1-Pad115)
- J1 pad 117: USB3-1-DP -> unconnected-(J1-Pad117)
- J1 pad 120: CSI-1_PWDN -> unconnected-(J1-Pad120)
- J1 pad 143: unconnected-(J1-Pad143) -> CAN_RX_(pin143_jet)
- J1 pad 145: unconnected-(J1-Pad145) -> CAN_TX_(pin145_jet)
- J1 pad 15: dCSI-0_D3_N -> CSI-0_D3_N
- J1 pad 17: dCSI-0_D3_P -> CSI-0_D3_P
- J1 pad 179: unconnected-(J1-Pad179) -> PCIe_WAKE_N
- J1 pad 21: dCSI-1_D2_N -> unconnected-(J1A-CSI3_D0_N-Pad21)
- J1 pad 22: dCSI-1_D0_N -> unconnected-(J1A-CSI2_D0_N-Pad22)
- J1 pad 23: dCSI-1_D2_P -> unconnected-(J1A-CSI3_D0_P-Pad23)
- J1 pad 24: dCSI-1_D0_P -> unconnected-(J1A-CSI2_D0_P-Pad24)
- J1 pad 28: dCSI-1_CLK_N -> unconnected-(J1A-CSI2_CLK_N-Pad28)
- J1 pad 3: dCSI-0_D2_N -> CSI-0_D2_N
- J1 pad 30: dCSI-1_CLK_P -> unconnected-(J1A-CSI2_CLK_P-Pad30)
- J1 pad 33: dCSI-1_D3_N -> unconnected-(J1A-CSI3_D1_N-Pad33)
- J1 pad 34: dCSI-1_D1_N -> unconnected-(J1A-CSI2_D1_N-Pad34)
- J1 pad 35: dCSI-1_D3_P -> unconnected-(J1A-CSI3_D1_P-Pad35)
- J1 pad 36: dCSI-1_D1_P -> unconnected-(J1A-CSI2_D1_P-Pad36)
- J1 pad 39: USB3-1-RX_N -> unconnected-(J1B-USBSS1_RX_N-Pad39)
- J1 pad 41: USB3-1-RX_P -> unconnected-(J1B-USBSS1_RX_P-Pad41)
- J1 pad 45: USB3-1-TX_N -> unconnected-(J1B-USBSS1_TX_N-Pad45)
- J1 pad 47: USB3-1-TX_P -> unconnected-(J1B-USBSS1_TX_P-Pad47)
- J1 pad 5: dCSI-0_D2_P -> CSI-0_D2_P
- Module1 pad 104: unconnected-(Module1-PCIe_nWAKE-Pad104) -> PCIe_WAKE_N
- Module1 pad 128: USB3-0-RX_N -> unconnected-(Module1-CAM0_D0_N-Pad128)
- Module1 pad 130: USB3-0-RX_P -> unconnected-(Module1-CAM0_D0_P-Pad130)
- Module1 pad 134: USB3-0-DP -> unconnected-(Module1-CAM0_D1_N-Pad134)
- Module1 pad 136: USB3-0-DN -> unconnected-(Module1-CAM0_D1_P-Pad136)
- Module1 pad 140: USB3-0-TX_N -> unconnected-(Module1-CAM0_CLK_N-Pad140)
- Module1 pad 142: USB3-0-TX_P -> unconnected-(Module1-CAM0_CLK_P-Pad142)
- Module1 pad 157: USB3-1-RX_N -> unconnected-(Module1-USB3-1-RX_N-Pad157)
- Module1 pad 159: USB3-1-RX_P -> unconnected-(Module1-USB3-1-RX_P-Pad159)
- Module1 pad 163: USB3-1-DP -> unconnected-(Module1-USB3-1-DP-Pad163)
- Module1 pad 165: USB3-1-DN -> unconnected-(Module1-USB3-1-DN-Pad165)
- Module1 pad 169: USB3-1-TX_N -> unconnected-(Module1-USB3-1-TX_N-Pad169)
- Module1 pad 171: USB3-1-TX_P -> unconnected-(Module1-USB3-1-TX_P-Pad171)
- R22 pad 1: HDMI-0_CLK_N -> +3V3
- R22 pad 2: dHDMI-0_CLK_N -> unconnected-(R22-Pad2)
- R23 pad 1: HDMI-0_CLK_P -> +3V3
- R23 pad 2: dHDMI-0_CLK_P -> unconnected-(R23-Pad2)
- U1 pad 1: +1V8 -> unconnected-(U1-USBDM_DN1/PRT_DIS_M1-Pad1)
- U1 pad 10: SPI-1_CS0_1V8 -> +3V3
- U1 pad 11: GND -> unconnected-(U1-TEST-Pad11)
- U1 pad 12: GND -> unconnected-(U1-PRTPWR1/BC_EN1-Pad12)
- U1 pad 13: GND -> unconnected-(U1-OCS_N1-Pad13)
- U1 pad 14: dSPI-1_CS0_3V3 -> Net-(U1-CRFILT)
- U1 pad 15: dSPI-1_CS1_3V3 -> +3V3
- U1 pad 16: dSPI-1_MOSI_3V3 -> unconnected-(U1-PRTPWR2/BC_EN2-Pad16)
- U1 pad 17: dSPI-1_CLK_3V3 -> unconnected-(U1-OCS_N2-Pad17)
- U1 pad 18: dSPI-0_CS1_3V3 -> unconnected-(U1-PRTPWR3/BC_EN3-Pad18)
- U1 pad 19: dSPI-0_CS0_3V3 -> unconnected-(U1-OCS_N3-Pad19)
- U1 pad 2: Net-(U1-DIR) -> unconnected-(U1-USBDP_DN1/PRT_DIS_P1-Pad2)
- U1 pad 20: dSPI-0_CLK_3V3 -> unconnected-(U1-PRTPWR4/BC_EN4-Pad20)
- U1 pad 21: dSPI-0_MOSI_3V3 -> unconnected-(U1-OCS_N4-Pad21)
- U1 pad 22: Net-(U1-~{OE}) -> unconnected-(U1-SDA/SMBDATA/NON_REM1-Pad22)
- U1 pad 24: +3V3 -> unconnected-(U1-SCL/SMBCLK/CFG_SEL0-Pad24)
- U1 pad 3: SPI-0_MOSI_1V8 -> unconnected-(U1-USBDM_DN2/PRT_DIS_M2-Pad3)
- U1 pad 4: SPI-0_CLK_1V8 -> unconnected-(U1-USBDP_DN2/PRT_DIS_P2-Pad4)
- U1 pad 5: SPI-0_CS0_1V8 -> +3V3
- U1 pad 6: SPI-0_CS1_1V8 -> unconnected-(U1-USBDM_DN3/PRT_DIS_M3-Pad6)
- U1 pad 7: SPI-1_CLK_1V8 -> unconnected-(U1-USBDP_DN3/PRT_DIS_P3-Pad7)
- U1 pad 8: SPI-1_MOSI_1V8 -> unconnected-(U1-USBDM_DN4/PRT_DIS_M4-Pad8)
- U1 pad 9: SPI-1_CS1_1V8 -> unconnected-(U1-USBDP_DN4/PRT_DIS_P4-Pad9)
Routing:
- net GND: track 196.8 -> 326.8 mm, vias 174 -> 200
- net (no net): track 0.00 -> 115.4 mm, vias 0 -> 4
- net unconnected-(J1-Pad104): track 0.00 -> 50.0 mm, vias 0 -> 2
- net SPI-1_MOSI_1V8: track 50.0 -> 0.00 mm, vias 2 -> 0
- net USB3-1-RX_P: track 48.1 -> 0.00 mm, vias 1 -> 0
- net USB3-1-RX_N: track 47.6 -> 0.00 mm
- net USB3-1-TX_P: track 45.5 -> 0.00 mm, vias 1 -> 0
- net USB3-1-TX_N: track 44.9 -> 0.00 mm
- net unconnected-(J1-Pad106): track 0.00 -> 44.2 mm, vias 0 -> 2
- net SPI-1_CLK_1V8: track 44.2 -> 0.00 mm, vias 2 -> 0
- net unconnected-(J1-Pad110): track 0.00 -> 40.6 mm, vias 0 -> 3
- net SPI-1_CS0_1V8: track 40.6 -> 0.00 mm, vias 3 -> 0
- net unconnected-(J1-Pad112): track 0.00 -> 39.6 mm, vias 0 -> 3
- net SPI-1_CS1_1V8: track 39.6 -> 0.00 mm, vias 3 -> 0
- net USB3-0-DN: track 12.3 -> 0.00 mm, vias 3 -> 0
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