File: PCB/cm4-high-speed.kicad_sch (KiCad schematic)
At the start: 1 part

Commit message: updated 2
Connections:
- net HDMI-0_CEC: now also Module1.149 (HDMI1_CEC); no longer Module1.151 (HDMI0_CEC)
- net CSI-1_D2_N: no longer names the net of Module1.193 (CSI1_D2_N)
- net CSI-1_D2_P: no longer names the net of Module1.195 (CSI1_D2_P)
- net CSI-1_D3_N: no longer names the net of Module1.194 (CSI1_D3_N)
- net CSI-1_D3_P: no longer names the net of Module1.196 (CSI1_D3_P)
- no-connect marks 16 -> 4
Other:
- note added: "0 USB3.0"
- note added: "1 USB3.0"
- note added: "CAMERA0"
- note added: "CAMERA1"
- note added: "CSI-(CAMERA NOTES)"
- note added: "CSI-2 differential pairs (the data path) 1x Clock lane: CLKP / CLKN 1 to 4x Data lanes: D0P/D0N, D1P/D1N, D2P/D2N, D3P/D3N"
- note added: "HDMI-Not needed"
- note added: "PCIE"
- note added: "SCL / SDA"
