File: PCB/cm4-high-speed.kicad_sch (KiCad schematic)
At the start: 1 part

Commit message: Fix broken CM4IO/SODIMM library links and add missing footprints
Both fp-lib-table and sym-lib-table pointed to other collaborators'
absolute local paths (a Windows user path and a Linux path), so the
CM4IO and SODIMM libraries could not resolve on this machine at all.
Repointed both tables at the project's own libraries/ folder using
${KIPRJMOD}-relative paths.

- Added the missing SODIMM_DDR4_EDGE footprint (260-pin card edge)
  and split the combined CM4 mezzanine footprint into
  Raspberry-Pi-4-Compute-Module-A/-B to match the schematic's
  existing per-connector pin numbering (1-100 / 101-200)
- Added Connectors.pretty and MCP25625T_E_ML.pretty footprint
  libraries that were referenced but never committed
- Moved the Mezzanine_A/Mezzanine_B symbols out of the orphaned
  "kai-library" reference (which pointed to no actual file) into
  the existing CM4IO symbol library
- Corrected Module1/Module2 MPN/Digi-Key part numbers to the
  primary DF40HC(3.0)-100DS-0.4V variant, keeping the old
  DF40C-100DS-0.4V values as (Alt) fields
- Reverted an in-progress SO-DIMM.kicad_sch rework that had
  misrouted 8 PCIe signals to the wrong physical pins and silently
  disconnected the CSI/USB3 nets, restoring the known-good pinout
  while keeping the CM4IO footprint rename

Co-Authored-By: Claude Sonnet 5 <noreply@anthropic.com>
Parts:
- Module1: footprint kai's library:Raspberry-Pi-4-Compute-Module-B -> CM4IO:Raspberry-Pi-4-Compute-Module-B; symbol kai-library:Mezzanine_B -> CM4IO:Mezzanine_B; Digi-Key_PN 2x H11615CT-ND -> 2x H124602CT-ND; Digi-Key_PN (Alt) 2x H124602CT-ND -> 2x H11615CT-ND; MPN 2x DF40C-100DS-0.4V -> 2x DF40HC(3.0)-100DS-0.4V; MPN (Alt) 2x DF40HC(3.0)-100DS-0.4V -> 2x DF40C-100DS-0.4V
Changed lines of the file:
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@@
 	)
 	(symbol
-		(lib_id "kai-library:Mezzanine_B")
+		(lib_id "CM4IO:Mezzanine_B")
 		(at 137.16 95.25 0)
 		(unit 1)
@@
 			)
 		)
-		(property "Footprint" "kai's library:Raspberry-Pi-4-Compute-Module-B"
+		(property "Footprint" "CM4IO:Raspberry-Pi-4-Compute-Module-B"
 			(at 279.4 121.92 0)
 			(hide yes)
@@
 			)
 		)
-		(property "MPN" "2x DF40C-100DS-0.4V"
+		(property "MPN" "2x DF40HC(3.0)-100DS-0.4V"
 			(at 137.922 23.622 0)
 			(show_name no)
@@
 			)
 		)
-		(property "Digi-Key_PN" "2x H11615CT-ND"
+		(property "Digi-Key_PN" "2x H124602CT-ND"
 			(at 137.668 35.306 0)
 			(hide yes)
@@
 			)
 		)
-		(property "MPN (Alt)" "2x DF40HC(3.0)-100DS-0.4V"
+		(property "MPN (Alt)" "2x DF40C-100DS-0.4V"
 			(at 137.922 26.162 0)
 			(show_name no)
@@
 			)
 		)
-		(property "Digi-Key_PN (Alt)" "2x H124602CT-ND"
+		(property "Digi-Key_PN (Alt)" "2x H11615CT-ND"
 			(at 137.668 33.274 0)
 			(hide yes)

Commit message: Add CAN/PCIe wake signals, drop USB3/CSI-1/most of SPI-1, route GbE pairs
Schematic changes (confirmed intentional):
- Renamed dCSI-0_D2/D3_N/P to CSI-0_D2/D3_N/P (same pins, label cleanup)
- Added CAN_RX/CAN_TX on J1 pins 143/145
- Added PCIe_WAKE_N on J1 pin 179 / Module1 pin 104 (repurposed from
  SPI-1_MOSI_1V8)
- Removed USB3-0 and USB3-1 (both ports entirely), the second CSI
  camera interface (dCSI-1, 10 signals), the remaining 4 SPI-1
  signals, and CSI-0/CSI-1_PWDN

PCB changes:
- Added carrier.kicad_dru with GbE differential pair rules: intra-pair
  skew <=0.25mm (1000BASE-T MDI tolerance) and inter-pair length
  matched to 49.7-50.7mm, both validated against kicad-cli pcb drc
- In-progress length tuning on the 4 GBE_MDI differential pairs

Co-Authored-By: Claude Sonnet 5 <noreply@anthropic.com>
Connections:
- net PCIe_WAKE_N: now reaches Module1.104 (PCIe_nWAKE)
- net USB3-0-DN: no longer names the net of Module1.136 (CAM0_D1_P)
- net USB3-0-DP: no longer names the net of Module1.134 (CAM0_D1_N)
- net USB3-0-RX_N: no longer names the net of Module1.128 (CAM0_D0_N)
- net USB3-0-RX_P: no longer names the net of Module1.130 (CAM0_D0_P)
- net USB3-0-TX_N: no longer names the net of Module1.140 (CAM0_CLK_N)
- net USB3-0-TX_P: no longer names the net of Module1.142 (CAM0_CLK_P)
- net USB3-1-DN: no longer names the net of Module1.165 (USB3-1-DN)
- net USB3-1-DP: no longer names the net of Module1.163 (USB3-1-DP)
- net USB3-1-RX_N: no longer names the net of Module1.157 (USB3-1-RX_N)
- net USB3-1-RX_P: no longer names the net of Module1.159 (USB3-1-RX_P)
- net USB3-1-TX_N: no longer names the net of Module1.169 (USB3-1-TX_N)
- net USB3-1-TX_P: no longer names the net of Module1.171 (USB3-1-TX_P)
