File: PCB/damping-resistors.kicad_sch (KiCad schematic)
At the start: 40 parts

Commit message: updated 2
Parts:
- removed R22, R23, R28, R29, R30, R31, R32, R33: 0, Resistor_SMD:R_0402_1005Metric, symbol Device:R
