File: PCB/level-shifting.kicad_sch (KiCad schematic)
At the start: 21 parts, among them U1 SN74LVC8T245, U2 SN74LVC8T245, U3 SN74LVC8T245

Commit message: Fix broken CM4IO/SODIMM library links and add missing footprints
Both fp-lib-table and sym-lib-table pointed to other collaborators'
absolute local paths (a Windows user path and a Linux path), so the
CM4IO and SODIMM libraries could not resolve on this machine at all.
Repointed both tables at the project's own libraries/ folder using
${KIPRJMOD}-relative paths.

- Added the missing SODIMM_DDR4_EDGE footprint (260-pin card edge)
  and split the combined CM4 mezzanine footprint into
  Raspberry-Pi-4-Compute-Module-A/-B to match the schematic's
  existing per-connector pin numbering (1-100 / 101-200)
- Added Connectors.pretty and MCP25625T_E_ML.pretty footprint
  libraries that were referenced but never committed
- Moved the Mezzanine_A/Mezzanine_B symbols out of the orphaned
  "kai-library" reference (which pointed to no actual file) into
  the existing CM4IO symbol library
- Corrected Module1/Module2 MPN/Digi-Key part numbers to the
  primary DF40HC(3.0)-100DS-0.4V variant, keeping the old
  DF40C-100DS-0.4V values as (Alt) fields
- Reverted an in-progress SO-DIMM.kicad_sch rework that had
  misrouted 8 PCIe signals to the wrong physical pins and silently
  disconnected the CSI/USB3 nets, restoring the known-good pinout
  while keeping the CM4IO footprint rename

Co-Authored-By: Claude Sonnet 5 <noreply@anthropic.com>
Parts:
- removed C10, C14, C17, C3: 0.1uF, Capacitor_SMD:C_0402_1005Metric, symbol Device:C
- removed C12, C16, C8, C9: 1uF, Capacitor_SMD:C_0402_1005Metric, symbol Device:C
- removed R2, R5, R6, R7: 10K, Resistor_SMD:R_0402_1005Metric, symbol Device:R
- removed U1, U3: SN74LVC8T245, Package_SO:TSSOP-24_4.4x5mm_P0.4mm, symbol Logic_LevelTranslator:SN74LVC8T245
Other:
- note removed: "Receive SPI/UART/TACH"
- note removed: "TRANSMIT SPI"
